File: PCB/KiCad project/KiCad project.kicad_pcb (KiCad board)
At the start: 2 copper layers, 42.9 x 62.4 mm, 7 parts, among them SW1 SW_Push, SW2 SW_Push, SW3 SW_Push, SW4 SW_Push, U1 XIAO-RP2040-DIP

Commit message: Add files via upload
Parts:
- added J1: Conn_01x04, Connector_PinHeader_2.54mm:PinHeader_1x04_P2.54mm_Vertical, F.Cu at (133.3, 52.1)
Connections:
- U1 pad 6: unconnected-(U1-GPIO7/SCL-Pad6) -> Net-(J1-Pin_3)
Routing:
- net Net-(J1-Pin_3): track 0.00 -> 11.9 mm, vias 0 -> 2
- net Net-(D1-DIN): track 5.48 -> 16.7 mm, vias 0 -> 2
