File: PCB/KiCad project/KiCad project.kicad_pcb (KiCad board)
At the start: 2 copper layers, 69.1 x 74.3 mm, 7 parts, among them SW2 SW_Push, SW3 SW_Push, SW4 SW_Push, U1 XIAO-RP2040-DIP, U2 OLED_0.91_128x32

Commit message: Add files via upload
Changed lines of the file:
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@@
+	)
+	(gr_rect
+		(start 175.26 90.17)
+		(end 185.07 90.17)
+		(stroke
+			(width 0.1)
+			(type default)
+		)
+		(fill no)
+		(layer "F.SilkS")
+	)
+	(gr_rect
+		(start 175.26 63.5)
+		(end 185.42 63.5)
+		(stroke
+			(width 0.1)
+			(type default)
+		)
+		(fill no)
+		(layer "F.SilkS")
 	)
 	(gr_rect

Commit message: Add files via upload
Parts:
- moved SW3 1.47 mm to (135.0, 97.6)
- moved SW4 1.10 mm to (155.1, 97.6)
- moved SW2 0.25 mm to (146.3, 77.5)
Connections:
- U1 pad 12: unconnected-(U1-3V3-Pad12) -> Net-(U1-3V3)
- U1 pad 4: unconnected-(U1-GPIO29/ADC3/A3-Pad4) -> Net-(D1-DIN)
- U1 pad 5: Net-(D1-DIN) -> Net-(U1-GPIO6/SDA)
- U1 pad 7: Net-(U1-GPIO0/TX) -> unconnected-(U1-GPIO0/TX-Pad7)
- U2 pad 2: +5V -> Net-(U1-3V3)
- U2 pad 4: Net-(U1-GPIO0/TX) -> Net-(U1-GPIO6/SDA)
Routing:
- net Net-(U1-GPIO0/TX): track 53.3 -> 0.00 mm, vias 2 -> 0
- net Net-(U1-GPIO6/SDA): track 0.00 -> 52.6 mm
- net +5V: track 61.6 -> 38.0 mm
- net Net-(U1-3V3): track 0.00 -> 21.9 mm, vias 0 -> 2
- net Net-(D1-DIN): track 11.3 -> 10.3 mm
- net (no net): track 0.00 -> 0.17 mm, vias 0 -> 1
Changed lines of the file:
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@@
 	(net 7 "Net-(U1-GPIO3{slash}MOSI)")
 	(net 8 "unconnected-(U1-GPIO28{slash}ADC2{slash}A2-Pad3)")
-	(net 9 "unconnected-(U1-3V3-Pad12)")
-	(net 10 "unconnected-(U1-GPIO29{slash}ADC3{slash}A3-Pad4)")
+	(net 9 "Net-(U1-3V3)")
+	(net 10 "Net-(U1-GPIO6{slash}SDA)")
 	(net 11 "unconnected-(U1-GPIO27{slash}ADC1{slash}A1-Pad2)")
 	(net 12 "unconnected-(U1-GPIO26{slash}ADC0{slash}A0-Pad1)")
 	(net 13 "unconnected-(U1-GPIO1{slash}RX-Pad8)")
-	(net 14 "Net-(U1-GPIO0{slash}TX)")
+	(net 14 "unconnected-(U1-GPIO0{slash}TX-Pad7)")
 	(net 15 "Net-(U1-GPIO7{slash}SCL)")
 	(net 16 "Net-(D1-DOUT)")
 	(footprint "Button_Switch_Keyboard:SW_Cherry_MX_1.00u_PCB"
 		(layer "F.Cu")
-		(at 146.05 77.47)
+		(at 146.3 77.48)
 		(descr "Cherry MX keyswitch, 1.00u, PCB mount, http://cherryamericas.com/wp-content/uploads/2014/12/mx_cat.pdf")
 		(tags "Cherry MX keyswitch 1.00u PCB")
@@
 			(layers "F.Cu" "F.Mask")
 			(roundrect_rratio 0.1)
-			(net 10 "unconnected-(U1-GPIO29{slash}ADC3{slash}A3-Pad4)")
+			(net 1 "Net-(D1-DIN)")
 			(pinfunction "GPIO29/ADC3/A3")
 			(pintype "passive")
@@
 			(layers "*.Cu" "*.Mask")
 			(remove_unused_layers no)
-			(net 10 "unconnected-(U1-GPIO29{slash}ADC3{slash}A3-Pad4)")
+			(net 1 "Net-(D1-DIN)")
 			(pinfunction "GPIO29/ADC3/A3")
 			(pintype "passive")
@@
 			(layers "F.Cu" "F.Mask")
 			(roundrect_rratio 0.1)
-			(net 1 "Net-(D1-DIN)")
+			(net 10 "Net-(U1-GPIO6{slash}SDA)")
 			(pinfunction "GPIO6/SDA")
 			(pintype "passive")
@@
 			(layers "*.Cu" "*.Mask")
 			(remove_unused_layers no)
-			(net 1 "Net-(D1-DIN)")
+			(net 10 "Net-(U1-GPIO6{slash}SDA)")
 			(pinfunction "GPIO6/SDA")
 			(pintype "passive")
@@
 			(layers "F.Cu" "F.Mask")
 			(roundrect_rratio 0.1)
-			(net 14 "Net-(U1-GPIO0{slash}TX)")
+			(net 14 "unconnected-(U1-GPIO0{slash}TX-Pad7)")
 			(pinfunction "GPIO0/TX")
 			(pintype "passive")
@@
 			(layers "*.Cu" "*.Mask")
 			(remove_unused_layers no)
-			(net 14 "Net-(U1-GPIO0{slash}TX)")
+			(net 14 "unconnected-(U1-GPIO0{slash}TX-Pad7)")
 			(pinfunction "GPIO0/TX")
 			(pintype "passive")
@@
 			(layers "*.Cu" "*.Mask")
 			(remove_unused_layers no)
-			(net 9 "unconnected-(U1-3V3-Pad12)")
+			(net 9 "Net-(U1-3V3)")
 			(pinfunction "3V3")
 			(pintype "passive")
@@
 			(layers "F.Cu" "F.Mask")
 			(roundrect_rratio 0.1)
-			(net 9 "unconnected-(U1-3V3-Pad12)")
+			(net 9 "Net-(U1-3V3)")
 			(pinfunction "3V3")
 			(pintype "passive")
@@
 	(footprint "Button_Switch_Keyboard:SW_Cherry_MX_1.00u_PCB"
 		(layer "F.Cu")
-		(at 155.019375 96.52)
+		(at 155.05 97.62)
 		(descr "Cherry MX keyswitch, 1.00u, PCB mount, http://cherryamericas.com/wp-content/uploads/2014/12/mx_cat.pdf")
 		(tags "Cherry MX keyswitch 1.00u PCB")
@@
 	(footprint "Button_Switch_Keyboard:SW_Cherry_MX_1.00u_PCB"
 		(layer "F.Cu")
-		(at 135.969375 96.52)
+		(at 134.98 97.61)
 		(descr "Cherry MX keyswitch, 1.00u, PCB mount, http://cherryamericas.com/wp-content/uploads/2014/12/mx_cat.pdf")
 		(tags "Cherry MX keyswitch 1.00u PCB")
@@
 			(layers "*.Cu" "*.Mask")
 			(remove_unused_layers no)
-			(net 3 "+5V")
+			(net 9 "Net-(U1-3V3)")
 			(pinfunction "VCC")
 			(pintype "power_in")
@@
 			(layers "*.Cu" "*.Mask")
 			(remove_unused_layers no)
-			(net 14 "Net-(U1-GPIO0{slash}TX)")
+			(net 10 "Net-(U1-GPIO6{slash}SDA)")
 			(pinfunction "SDA")
 			(pintype "bidirectional")
@@
 	)
 	(segment
+		(start 163.83 40.92)
+		(end 163.83 40.7542)
+		(width 0.2)
+		(layer "F.Cu")
+		(net 0)
+	)
+	(via
+		(at 163.83 40.7542)
+		(size 0.6)
+		(drill 0.3)
+		(layers "F.Cu" "B.Cu")
+		(net 0)
+	)
+	(segment
+		(start 141.7795 46.99)
+		(end 145.215 50.4255)
+		(width 0.2)
+		(layer "F.Cu")
+		(net 1)
+	)
+	(segment
 		(start 136.37 46.99)
-		(end 139.2395 46.99)
-		(width 0.2)
-		(layer "F.Cu")
-		(net 1)
-	)
-	(segment
-		(start 139.2395 46.99)
-		(end 145.215 52.9655)
+		(end 141.7795 46.99)
 		(width 0.2)
 		(layer "F.Cu")
@@
 	)
 	(segment
-		(start 177.8 58.4805)
-		(end 162.125 42.8055)
-		(width 0.2)
-		(layer "F.Cu")
-		(net 3)
-	)
-	(segment
 		(start 140.97 40.64)
 		(end 159.9595 40.64)
@@
 	)
 	(segment
-		(start 177.8 59.97)
-		(end 177.8 58.4805)
-		(width 0.2)
-		(layer "F.Cu")
-		(net 3)
-	)
-	(segment
 		(start 144.78 72.39)
 		(end 154.94 62.23)
@@
 	)
 	(segment
-		(start 139.7 80.01)
-		(end 139.7 77.47)
+		(start 140 80.02)
+		(end 140 77.48)
 		(width 0.2)
 		(layer "F.Cu")
@@
 	)
 	(segment
-		(start 139.7 77.47)
-		(end 142.24 74.93)
+		(start 140 77.48)
+		(end 142.54 74.94)
 		(width 0.2)
 		(layer "F.Cu")
@@
 	)
 	(via
-		(at 144.78 72.39)
+		(at 145.08 72.4)
 		(size 0.6)
 		(drill 0.3)
@@
 	)
 	(via
-		(at 142.24 74.93)
+		(at 142.54 74.94)
 		(size 0.6)
 		(drill 0.3)
@@
 	)
 	(segment
-		(start 142.24 74.93)
-		(end 144.78 72.39)
+		(start 142.54 74.94)
+		(end 145.08 72.4)
 		(width 0.2)
 		(layer "B.Cu")
@@
 	)
 	(segment
-		(start 182.88 59.97)
-		(end 163.83 40.92)
-		(width 0.2)
-		(layer "F.Cu")
-		(net 14)
-	)
-	(segment
-		(start 158.75 45.3455)
-		(end 146.05 58.0455)
-		(width 0.2)
-		(layer "F.Cu")
-		(net 14)
-	)
-	(segment
-		(start 163.83 40.92)
-		(end 163.83 40.7542)
-		(width 0.2)
-		(layer "F.Cu")
-		(net 14)
-	)
-	(segment
-		(start 158.75 43.18)
-		(end 158.75 45.3455)
-		(width 0.2)
-		(layer "F.Cu")
-		(net 14)
+		(start 163.83 48.26)
+		(end 162.4995 48.26)
+		(width 0.2)
+		(layer "F.Cu")
+		(net 9)
+	)
+	(segment
+		(start 177.8 59.97)
+		(end 165.1 47.27)
+		(width 0.2)
+		(layer "F.Cu")
+		(net 9)
+	)
+	(segment
+		(start 165.1 47.27)
+		(end 165.1 46.99)
+		(width 0.2)
+		(layer "F.Cu")
+		(net 9)
+	)
+	(segment
+		(start 162.4995 48.26)
+		(end 162.125 47.8855)
+		(width 0.2)
+		(layer "F.Cu")
+		(net 9)
 	)
 	(via
-		(at 163.83 40.7542)
+		(at 163.83 48.26)
 		(size 0.6)
 		(drill 0.3)
 		(layers "F.Cu" "B.Cu")
-		(net 14)
+		(net 9)
 	)
 	(via
-		(at 158.75 43.18)
+		(at 165.1 46.99)
 		(size 0.6)
 		(drill 0.3)
 		(layers "F.Cu" "B.Cu")
-		(net 14)
-	)
-	(segment
-		(start 163.229 41.3552)
-		(end 160.5748 41.3552)
+		(net 9)
+	)
+	(segment
+		(start 165.1 46.99)
+		(end 163.83 48.26)
 		(width 0.2)
 		(layer "B.Cu")
-		(net 14)
-	)
-	(segment
-		(start 163.83 40.7542)
-		(end 163.229 41.3552)
-		(width 0.2)
-		(layer "B.Cu")
-		(net 14)
-	)
-	(segment
-		(start 160.5748 41.3552)
-		(end 158.75 43.18)
-		(width 0.2)
-		(layer "B.Cu")
-		(net 14)
-	)
-	(segment
+		(net 9)
+	)
+	(segment
+		(start 161.14764 49.24645)
+		(end 158.081 46.17981)
+		(width 0.2)
+		(layer "F.Cu")
+		(net 10)
+	)
+	(segment
+		(start 182.88 59.97)
+		(end 181.729 61.121)
+		(width 0.2)
+		(layer "F.Cu")
+		(net 10)
+	)
+	(segment
+		(start 174.109 59.809)
+		(end 163.54645 49.24645)
+		(width 0.2)
+		(layer "F.Cu")
+		(net 10)
+	)
+	(segment
+		(start 174.109 60.849804)
+		(end 174.109 59.809)
+		(width 0.2)
+		(layer "F.Cu")
+		(net 10)
+	)
+	(segment
+		(start 158.081 46.17981)
+		(end 158.081 42.931057)
+		(width 0.2)
+		(layer "F.Cu")
+		(net 10)
+	)
+	(segment
+		(start 155.6015 42.579)
+		(end 145.215 52.9655)
+		(width 0.2)
+		(layer "F.Cu")
+		(net 10)
+	)
+	(segment
+		(start 174.380196 61.121)
+		(end 174.109 60.849804)
+		(width 0.2)
+		(layer "F.Cu")
+		(net 10)
+	)
+	(segment
+		(start 158.081 42.931057)
+		(end 157.728943 42.579)
+		(width 0.2)
+		(layer "F.Cu")
+		(net 10)
+	)
+	(segment
+		(start 181.729 61.121)
+		(end 174.380196 61.121)
+		(width 0.2)
+		(layer "F.Cu")
+		(net 10)
+	)
+	(segment
+		(start 163.54645 49.24645)
+		(end 161.14764 49.24645)
+		(width 0.2)
+		(layer "F.Cu")
+		(net 10)
+	)
+	(segment
+		(start 157.728943 42.579)
+		(end 155.6015 42.579)
+		(width 0.2)
+		(layer "F.Cu")
+		(net 10)
+	)
+	(segment

Commit message: Add files via upload
Parts:
- removed D1, D2: SK6812MINI, LED_SMD:LED_SK6812MINI_PLCC4_3.5x3.5mm_P1.75mm
- added D3: SK6812MINI-E, SK mini e:SK6812MINI-E_fixed, B.Cu at (134.0, 48.4)
- added D4: SK6812MINI-E, SK mini e:SK6812MINI-E_fixed, B.Cu at (134.0, 53.5)
- moved SW2 1.26 mm to (145.2, 76.9)
- moved SW4 0.73 mm to (155.2, 96.9)
- moved SW3 0.73 mm to (135.2, 96.9)
Routing:
- net Net-(D3-DIN): track 0.00 -> 17.7 mm
- net Net-(D1-DOUT): track 13.9 -> 0.00 mm, vias 2 -> 0
- net +5V: track 38.0 -> 46.6 mm, vias 0 -> 5
- net Net-(D4-DIN): track 10.3 -> 16.2 mm, vias 0 -> 2
- net GND: track 136.4 -> 137.1 mm
Other:
- board text removed: "1"
