File: PCB/KiCad project/KiCad project.kicad_pcb (KiCad board)
At the start: 2 copper layers, 69.1 x 74.3 mm, 7 parts, among them SW2 SW_Push, SW3 SW_Push, SW4 SW_Push, U1 XIAO-RP2040-DIP, U2 OLED_0.91_128x32

Commit message: Add files via upload
Parts:
- D3, D4: moved to F.Cu
- turned D3 to 0 degrees
- turned D4 to 0 degrees
Routing:
- net GND: track 137.1 -> 128.0 mm, vias 4 -> 2
- net Net-(D4-DIN): track 16.2 -> 9.49 mm, vias 2 -> 3
- net +5V: track 46.6 -> 41.1 mm, vias 5 -> 2
- net Net-(D3-DIN): track 17.7 -> 18.7 mm, vias 0 -> 2
Other:
- outline, holes or cut-outs redrawn
