File: PCB/KiCad project/KiCad project.kicad_sch (KiCad schematic)
At the start: 7 parts, among them SW2 SW_Push, SW3 SW_Push, SW4 SW_Push, U1 XIAO-RP2040-DIP, U2 OLED_0.91_128x32

Commit message: Add files via upload
Connections:
- net +5V: no longer U2.2 (VCC)
- net at U1.12 (3V3): now also U2.2 (VCC)
- net at U1.4 (GPIO29/ADC3/A3): now also D1.3 (DIN)
- net at U1.5 (GPIO6/SDA): now also U2.4 (SDA); no longer D1.3 (DIN)
- net at U1.7 (GPIO0/TX): no longer U2.4 (SDA)
Other:
- moved on the sheet: SW3, SW4
