File: PCB/KiCad project/_autosave-KiCad project.kicad_pcb (KiCad board)
At the start: 2 copper layers, 69.1 x 74.3 mm, 7 parts, among them SW2 SW_Push, SW3 SW_Push, SW4 SW_Push, U1 XIAO-RP2040-DIP, U2 OLED_0.91_128x32

Commit message: Add files via upload
Parts:
- removed D1, D2: SK6812MINI, LED_SMD:LED_SK6812MINI_PLCC4_3.5x3.5mm_P1.75mm
- added D3: SK6812MINI-E, SK mini e:SK6812MINI-E_fixed, F.Cu at (134.0, 48.4)
- added D4: SK6812MINI-E, SK mini e:SK6812MINI-E_fixed, F.Cu at (134.0, 53.5)
Routing:
- net Net-(D3-DIN): track 0.00 -> 18.7 mm, vias 0 -> 2
- net Net-(D1-DOUT): track 13.9 -> 0.00 mm, vias 2 -> 0
- net GND: track 136.4 -> 128.0 mm, vias 4 -> 2
- net +5V: track 38.0 -> 41.1 mm, vias 0 -> 2
- net Net-(D4-DIN): track 10.3 -> 9.49 mm, vias 0 -> 3
Other:
- outline, holes or cut-outs redrawn
- board text removed: "1"
